File: 20160111_scanimage-bias/scanimage-bias.brd (EAGLE design)
At the start: 65 x 40 mm, 16 parts

Commit message: ScanImage board WIP
Parts:
- moved J5 108.0 mm to (53.3, 29.8), turned to 180 degrees
- moved C8 91.0 mm to (57.1, 11.4), turned to 90 degrees
- moved C7 89.3 mm to (47.0, 21.6), turned to 90 degrees
- moved J4 75.5 mm to (50.8, 3.81)
- moved J3 67.4 mm to (27.9, 29.8), turned to 180 degrees
- moved C4 63.4 mm to (33.0, 17.8), turned to 90 degrees
- moved C6 63.1 mm to (5.16, 21.2)
- moved U$3 62.5 mm to (52.1, 15.2), turned to 90 degrees
- moved C5 62.3 mm to (16.6, 21.4)
- moved C1 50.5 mm to (41.3, 27.9), turned to 90 degrees
- moved C3 46.8 mm to (33.2, 8.97), turned to 90 degrees
- moved J2 41.2 mm to (25.4, 3.81)
- moved J1 40.9 mm to (11.4, 29.8), turned to 180 degrees
- moved C2 37.8 mm to (20.4, 14.1), turned to 90 degrees
- moved U$1 30.8 mm to (39.4, 19.1), turned to 270 degrees
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Routing:
- net VCC: track 0.00 -> 73.7 mm, vias 0 -> 1
- net VREF: track 0.00 -> 33.5 mm
- net OUT1: track 0.00 -> 21.0 mm
- net OUT2: track 0.00 -> 15.9 mm
- net VNEG: track 0.00 -> 9.64 mm
- added copper zone on layer 1, net GND
Other:
- board size 65 x 40 mm -> 65 x 33 mm

Commit message: Completed board -- rev1
Parts:
- moved C4 12.8 mm to (38.7, 6.35), turned to 270 degrees
- moved C1 8.64 mm to (38.7, 19.7), turned to 270 degrees
- moved C8 8.47 mm to (59.1, 19.7), turned to 270 degrees
- moved C6 7.70 mm to (12.7, 19.7), turned to 270 degrees
- moved C7 6.84 mm to (44.5, 15.2), turned to 180 degrees
- moved U$1 5.75 mm to (33.7, 18.4)
- moved C2 4.10 mm to (19.1, 10.2), turned to 180 degrees
- moved C3 2.65 mm to (33.7, 6.35)
- moved C5 2.52 mm to (18.4, 19.7), turned to 270 degrees
- moved J1 1.42 mm to (12.7, 29.2)
- moved J3 1.42 mm to (29.2, 29.2)
- moved J5 1.42 mm to (54.6, 29.2)
- moved J2 1.27 mm to (26.7, 3.81)
- moved J4 1.27 mm to (52.1, 3.81)
- moved U$3 1.27 mm to (53.3, 15.2)
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Routing:
- net VNEG: track 9.64 -> 94.0 mm, vias 0 -> 3
- net IN2: track 0.00 -> 11.1 mm
- net IN1: track 0.00 -> 6.03 mm
- net VCC: track 73.7 -> 79.2 mm, vias 1 -> 2
- net VREF: track 33.5 -> 38.6 mm, vias 0 -> 2
- net OUT1: track 21.0 -> 20.3 mm
- net OUT2: track 15.9 -> 15.2 mm
- added copper zone on layer 16, net GND
Other:
- board text added: "+12"
- board text added: "-12"
- board text added: "BIAS BOARD (2.5 V) 2016 JAN 14 KIMTH@STANFORD.EDU"
- board text added: "GND"
- board text added: "IN1"
- board text added: "IN2"
- board text added: "OUT1"
- board text added: "OUT2"
